File: FuenteBAE/FuenteBAE.kicad_sch (KiCad schematic)
At the start: 15 parts, among them J1 Screw_Terminal_01x02, J2 Screw_Terminal_01x02, U1 LM317_TO-220

Commit message: Add files via upload
Parts:
- C1: value C_Polarized -> 1000uF
- C2: value C_Polarized -> 10uF
- C3, C4: value C -> 0.1uF
- R1: value R -> 220Ohm
- R2: value R -> 1Kohm
- RV1: value R_Potentiometer -> 5Kohm
Changed lines of the file:
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@@
 			)
 		)
-		(property "Value" "C_Polarized"
+		(property "Value" "1000uF"
 			(at 124.46 93.0909 0)
 			(effects
@@
 			)
 		)
-		(property "Value" "R"
+		(property "Value" "220Ohm"
 			(at 179.07 93.9799 0)
 			(effects
@@
 			)
 		)
-		(property "Value" "R"
+		(property "Value" "1Kohm"
 			(at 238.76 88.8999 0)
 			(effects
@@
 			)
 		)
-		(property "Value" "C"
+		(property "Value" "0.1uF"
 			(at 196.85 106.6799 0)
 			(effects
@@
 			)
 		)
-		(property "Value" "C_Polarized"
+		(property "Value" "10uF"
 			(at 214.63 93.0909 0)
 			(effects
@@
 			)
 		)
-		(property "Value" "R_Potentiometer"
+		(property "Value" "5Kohm"
 			(at 162.56 120.6499 0)
 			(effects
@@
 			)
 		)
-		(property "Value" "C"
+		(property "Value" "0.1uF"
 			(at 148.59 106.6799 0)
 			(effects
